Commit message: 2.009 Update urdf to facilitate optional controls

File: panda_description/urdf/panda.urdf.xacro (robot description, xacro)
@@ -5,7 +5,8 @@
     <!-- Is the robot being simulated in gazebo?" -->
     <xacro:arg name="gazebo" default="true" />
+    <xacro:arg name="ros2_control" default="false" />
     <!-- Should a franka_gripper be mounted at the flange?" -->
     <xacro:arg name="hand" default="true" />
-  <xacro:panda_robot arm_id="$(arg arm_id)" joint_limits="${xacro.load_yaml('$(find panda_description)/config/joint_limits.yaml')}" hand="$(arg hand)" gazebo="$(arg gazebo)">
+  <xacro:panda_robot arm_id="$(arg arm_id)" joint_limits="${xacro.load_yaml('$(find panda_description)/config/joint_limits.yaml')}" hand="$(arg hand)" gazebo="$(arg gazebo)"  ros2_control="$(arg ros2_control)">
   </xacro:panda_robot>
 </robot>

File: panda_description/urdf/panda_robot.xacro (robot description, xacro)
@@ -1,5 +1,5 @@
 <?xml version='1.0' encoding='utf-8'?>
 <robot xmlns:xacro="http://www.ros.org/wiki/xacro">
-  <xacro:macro name="panda_robot" params="arm_id joint_limits hand gazebo">
+  <xacro:macro name="panda_robot" params="arm_id joint_limits hand gazebo ros2_control">
     <!-- Name of this panda -->
     <!-- Positional offset between $(arm_id)_hand -> $(arm_id)_hand_tcp [m]. Only used when hand:=true -->
@@ -54,9 +54,4 @@
       <xacro:gazebo-joint joint="${arm_id}_joint6" transmission="hardware_interface/EffortJointInterface" />
       <xacro:gazebo-joint joint="${arm_id}_joint7" transmission="hardware_interface/EffortJointInterface" />
-      <!-- <xacro:transmission-franka-state arm_id="${arm_id}" />
-      <xacro:transmission-franka-model arm_id="${arm_id}"
-         root="${arm_id}_joint1"
-         tip="${arm_id}_joint8"
-       /> -->
       <xacro:if value="$(arg hand)">
         <xacro:gazebo-joint joint="${arm_id}_finger_joint1" transmission="hardware_interface/EffortJointInterface" />
@@ -66,23 +61,25 @@
         <xacro:gazebo-friction link="${arm_id}_rightfinger" mu="1.13" />
       </xacro:if>
-     <ros2_control name="GazeboSystem" type="system">
-      <hardware>
-        <plugin>gazebo_ros2_control/GazeboSystem</plugin>
-      </hardware>
-        <xacro:ros2_control_joint joint="${arm_id}_joint1" />
-        <xacro:ros2_control_joint joint="${arm_id}_joint2" />
-        <xacro:ros2_control_joint joint="${arm_id}_joint3" />
-        <xacro:ros2_control_joint joint="${arm_id}_joint4" />
-        <xacro:ros2_control_joint joint="${arm_id}_joint5" />
-        <xacro:ros2_control_joint joint="${arm_id}_joint6" />
-        <xacro:ros2_control_joint joint="${arm_id}_joint7" />
-        <xacro:ros2_control_joint joint="${arm_id}_finger_joint1"/>
-        <xacro:ros2_control_joint joint="${arm_id}_finger_joint2"/>
-      </ros2_control>
-      <gazebo>
-        <plugin name="gazebo_ros2_control" filename="libgazebo_ros2_control.so">
-          <parameters>$(find panda_description)/config/controllers_effort.yaml</parameters>
-        </plugin>
-      </gazebo>
+      <xacro:if value="$(arg ros2_control)">
+        <ros2_control name="GazeboSystem" type="system">
+          <hardware>
+            <plugin>gazebo_ros2_control/GazeboSystem</plugin>
+          </hardware>
+            <xacro:ros2_control_joint joint="${arm_id}_joint1" />
+            <xacro:ros2_control_joint joint="${arm_id}_joint2" />
+            <xacro:ros2_control_joint joint="${arm_id}_joint3" />
+            <xacro:ros2_control_joint joint="${arm_id}_joint4" />
+            <xacro:ros2_control_joint joint="${arm_id}_joint5" />
+            <xacro:ros2_control_joint joint="${arm_id}_joint6" />
+            <xacro:ros2_control_joint joint="${arm_id}_joint7" />
+            <xacro:ros2_control_joint joint="${arm_id}_finger_joint1"/>
+            <xacro:ros2_control_joint joint="${arm_id}_finger_joint2"/>
+        </ros2_control>
+        <gazebo>
+          <plugin name="gazebo_ros2_control" filename="libgazebo_ros2_control.so">
+            <parameters>$(find panda_description)/config/controllers_effort.yaml</parameters>
+          </plugin>
+        </gazebo>
+      </xacro:if>
     </xacro:if>
   </xacro:macro>

File: panda_description/urdf/utils.xacro (robot description, xacro)
@@ -175,27 +175,4 @@
     </transmission>
   </xacro:macro>
-  <!-- ============================================================ -->
-  <!-- Adds the required tags to provide a `FrankaModelInterface`   -->
-  <!-- when simulating with franka_hw_sim plugin                    -->
-  <!--                                                              -->
-  <!-- arm_id - Arm ID of the panda to simulate (default 'panda')   -->
-  <!-- root   - Joint name of the base of the robot                 -->
-  <!-- tip    - Joint name of the tip of the robot (flange or hand) -->
-  <!-- ============================================================ -->
-  <xacro:macro name="transmission-franka-model" params="arm_id:=panda root:=panda_joint1 tip:=panda_joint7">
-    <transmission name="${arm_id}_franka_model">
-      <type>franka_hw/FrankaModelInterface</type>
-      <joint name="${root}">
-        <role>root</role>
-        <hardwareInterface>franka_hw/FrankaModelInterface</hardwareInterface>
-      </joint>
-      <joint name="${tip}">
-        <role>tip</role>
-        <hardwareInterface>franka_hw/FrankaModelInterface</hardwareInterface>
-      </joint>
-      <actuator name="${root}_motor_root"><hardwareInterface>franka_hw/FrankaModelInterface</hardwareInterface></actuator>
-      <actuator name="${tip}_motor_tip"  ><hardwareInterface>franka_hw/FrankaModelInterface</hardwareInterface></actuator>
-    </transmission>
-  </xacro:macro>
   <xacro:macro name="inertia-cylinder" params="mass radius h">
     <inertial>
@@ -238,5 +215,7 @@
           <command_interface name="effort"/>
         </xacro:if>
-        <state_interface name="position"/>
+        <state_interface name="position">
+            <param name="initial_value">0.0</param>
+        </state_interface>
         <state_interface name="velocity"/>
         <state_interface name="effort"/>

Commit message: 2.039, 2.040 Update the urdf of the hand and arm to allow of optional generation of collision models

File: panda_description/urdf/panda.urdf.xacro (robot description, xacro)
@@ -3,10 +3,13 @@
   <xacro:include filename="$(find panda_description)/urdf/panda_robot.xacro"/>
   <xacro:arg name="arm_id" default="panda" />
-    <!-- Is the robot being simulated in gazebo?" -->
-    <xacro:arg name="gazebo" default="true" />
-    <xacro:arg name="ros2_control" default="false" />
-    <!-- Should a franka_gripper be mounted at the flange?" -->
-    <xacro:arg name="hand" default="true" />
-  <xacro:panda_robot arm_id="$(arg arm_id)" joint_limits="${xacro.load_yaml('$(find panda_description)/config/joint_limits.yaml')}" hand="$(arg hand)" gazebo="$(arg gazebo)"  ros2_control="$(arg ros2_control)">
+  <!-- Is the robot being simulated in gazebo?" -->
+  <xacro:arg name="gazebo" default="true" />
+  <!-- Is the robot being using ros2_control?" -->
+  <xacro:arg name="ros2_control" default="false" />
+  <!-- Should the collision meshes be loaded?" -->
+  <xacro:arg name="collision_enable" default="true" />
+  <!-- Should a franka_gripper be mounted at the flange?" -->
+  <xacro:arg name="hand" default="true" />
+  <xacro:panda_robot arm_id="$(arg arm_id)" joint_limits="${xacro.load_yaml('$(find panda_description)/config/joint_limits.yaml')}" hand="$(arg hand)" gazebo="$(arg gazebo)" ros2_control="$(arg ros2_control)" collision_enable="$(arg collision_enable)">
   </xacro:panda_robot>
 </robot>

File: panda_description/urdf/panda_arm.xacro (robot description, xacro)
@@ -5,5 +5,5 @@
   <!-- arm_id: Namespace of the robot arm. Serves to differentiate between arms in case of multiple instances. -->
   <!-- joint_limits: description of the joint limits that comes from a YAML file. Example definition: ${xacro.load_yaml('$(find panda_description)/robots/fr3/joint_limits.yaml')} -->
-  <xacro:macro name="panda_arm" params="arm_id:='panda' description_pkg:='panda_description' connected_to:='' xyz:='0 0 0' rpy:='0 0 0' gazebo:=false safety_distance:=0 joint_limits" >
+  <xacro:macro name="panda_arm" params="arm_id:='panda' description_pkg:='panda_description' connected_to:='' xyz:='0 0 0' rpy:='0 0 0' gazebo:=false safety_distance:=0 joint_limits collision_enable:=true" >
     <xacro:unless value="${not connected_to}">
       <joint name="${arm_id}_joint_${connected_to}" type="fixed">
@@ -13,10 +13,10 @@
       </joint>
     </xacro:unless>
-    <xacro:link_with_sc name="link0" gazebo="${gazebo}">
+    <xacro:link_with_sc name="link0" gazebo="${gazebo}" collision_enable="${collision_enable}">
       <self_collision_geometries>
         <xacro:collision_capsule xyz="-0.075 0 0.06" direction="x" radius="${0.06+safety_distance}" length="0.03" />
       </self_collision_geometries>
     </xacro:link_with_sc>
-    <xacro:link_with_sc name="link1" gazebo="${gazebo}">
+    <xacro:link_with_sc name="link1" gazebo="${gazebo}" collision_enable="${collision_enable}">
       <self_collision_geometries>
         <xacro:collision_capsule xyz="0 0 -191.5e-3" radius="${0.06+safety_distance}" length="0.283" />
@@ -31,5 +31,5 @@
       <dynamics D="1" K="7000" damping="0.003" friction="0.0" mu_coulomb="0" mu_viscous="16" />
     </joint>
-    <xacro:link_with_sc name="link2" gazebo="${gazebo}">
+    <xacro:link_with_sc name="link2" gazebo="${gazebo}" collision_enable="${collision_enable}">
       <self_collision_geometries>
         <xacro:collision_capsule xyz="0 0 0" radius="${0.06+safety_distance}" length="0.12" />
@@ -44,5 +44,5 @@
       <dynamics D="1" K="7000" damping="0.003" friction="0.0" mu_coulomb="0" mu_viscous="16" />
     </joint>
-    <xacro:link_with_sc name="link3" gazebo="${gazebo}">
+    <xacro:link_with_sc name="link3" gazebo="${gazebo}" collision_enable="${collision_enable}">
       <self_collision_geometries>
         <xacro:collision_capsule xyz="0 0 -0.145" radius="${0.06+safety_distance}" length="0.15" />
@@ -57,5 +57,5 @@
       <dynamics D="1" K="7000" damping="0.003" friction="0.0" mu_coulomb="0" mu_viscous="16" />
     </joint>
-    <xacro:link_with_sc name="link4" gazebo="${gazebo}">
+    <xacro:link_with_sc name="link4" gazebo="${gazebo}" collision_enable="${collision_enable}">
       <self_collision_geometries>
         <xacro:collision_capsule xyz="0 0 0" radius="${0.06+safety_distance}" length="0.12" />
@@ -70,5 +70,5 @@
       <dynamics D="1" K="7000" damping="0.003" friction="0.0" mu_coulomb="0" mu_viscous="16" />
     </joint>
-    <xacro:link_with_sc name="link5" gazebo="${gazebo}">
+    <xacro:link_with_sc name="link5" gazebo="${gazebo}" collision_enable="${collision_enable}">
       <self_collision_geometries>
         <xacro:collision_capsule xyz="0 0 -0.26"    radius="${0.060+safety_distance}" length="0.10" />
@@ -84,5 +84,5 @@
       <dynamics D="1" K="7000" damping="0.003" friction="0.0" mu_coulomb="0" mu_viscous="16" />
     </joint>
-    <xacro:link_with_sc name="link6" gazebo="${gazebo}">
+    <xacro:link_with_sc name="link6" gazebo="${gazebo}" collision_enable="${collision_enable}">
       <self_collision_geometries>
         <xacro:collision_capsule xyz="0 0 -0.03" radius="${0.05+safety_distance}" length="0.08" />
@@ -97,5 +97,5 @@
       <dynamics D="1" K="7000" damping="0.003" friction="0.0" mu_coulomb="0" mu_viscous="16" />
     </joint>
-    <xacro:link_with_sc name="link7" gazebo="${gazebo}" rpy="0 0 ${pi/4}">
+    <xacro:link_with_sc name="link7" gazebo="${gazebo}" rpy="0 0 ${pi/4}" collision_enable="${collision_enable}">
       <self_collision_geometries>
         <xacro:collision_capsule xyz="0 0 0.01" direction="z" radius="${0.04+safety_distance}" length="0.14" />

File: panda_description/urdf/panda_hand.xacro (robot description, xacro)
@@ -2,5 +2,5 @@
 <robot xmlns:xacro="http://www.ros.org/wiki/xacro" name="hand">
   <!-- safety_distance: Minimum safety distance in [m] by which the collision volumes are expanded and which is enforced during robot motions -->
-  <xacro:macro name="panda_hand" params="connected_to:='' arm_id:='panda' rpy:='0 0 0' xyz:='0 0 0' tcp_xyz:='0 0 0.1034' tcp_rpy:='0 0 0' safety_distance:=0 gazebo:=false description_pkg:=panda_description">
+  <xacro:macro name="panda_hand" params="connected_to:='' arm_id:='panda' rpy:='0 0 0' xyz:='0 0 0' tcp_xyz:='0 0 0.1034' tcp_rpy:='0 0 0' safety_distance:=0 gazebo:=false description_pkg:=panda_description collision_enable:=true">
     <xacro:unless value="${connected_to == ''}">
       <joint name="${arm_id}_hand_joint" type="fixed">
@@ -10,5 +10,5 @@
       </joint>
     </xacro:unless>
-    <xacro:link_with_sc name="hand" gazebo="${gazebo}">
+    <xacro:link_with_sc name="hand" gazebo="${gazebo}" collision_enable="${collision_enable}">
       <self_collision_geometries>
         <xacro:collision_capsule xyz="0 0 0.04" direction="y" radius="${0.04+safety_distance}" length="0.1" />
@@ -29,25 +29,27 @@
         </geometry>
       </visual>
+      <xacro:if value="${collision_enable}">
       <!-- screw mount -->
-      <collision>
-        <origin xyz="0 18.5e-3 11e-3" rpy="0 0 0" />
-        <geometry>
-          <box size="22e-3 15e-3 20e-3" />
-        </geometry>
-      </collision>
-      <!-- cartriage sledge -->
-      <collision>
-        <origin xyz="0 6.8e-3 2.2e-3" rpy="0 0 0" />
-        <geometry>
-          <box size="22e-3 8.8e-3 3.8e-3" />
-        </geometry>
-      </collision>
-      <!-- diagonal finger -->
-      <collision>
-        <origin xyz="0 15.9e-3 28.35e-3" rpy="${pi/6} 0 0" />
-        <geometry>
-          <box size="17.5e-3 7e-3 23.5e-3" />
-        </geometry>
-      </collision>
+        <collision>
+          <origin xyz="0 18.5e-3 11e-3" rpy="0 0 0" />
+          <geometry>
+            <box size="22e-3 15e-3 20e-3" />
+          </geometry>
+        </collision>
+        <!-- cartriage sledge -->
+        <collision>
+          <origin xyz="0 6.8e-3 2.2e-3" rpy="0 0 0" />
+          <geometry>
+            <box size="22e-3 8.8e-3 3.8e-3" />
+          </geometry>
+        </collision>
+        <!-- diagonal finger -->
+        <collision>
+          <origin xyz="0 15.9e-3 28.35e-3" rpy="${pi/6} 0 0" />
+          <geometry>
+            <box size="17.5e-3 7e-3 23.5e-3" />
+          </geometry>
+        </collision>
+      </xacro:if>
       <!-- rubber tip with which to grasp -->
       <collision>
@@ -68,25 +70,27 @@
         </geometry>
       </visual>
-      <!-- screw mount -->
-      <collision>
-        <origin xyz="0 -18.5e-3 11e-3" rpy="0 0 0" />
-        <geometry>
-          <box size="22e-3 15e-3 20e-3" />
-        </geometry>
-      </collision>
-      <!-- cartriage sledge -->
-      <collision>
-        <origin xyz="0 -6.8e-3 2.2e-3" rpy="0 0 0" />
-        <geometry>
-          <box size="22e-3 8.8e-3 3.8e-3" />
-        </geometry>
-      </collision>
-      <!-- diagonal finger -->
-      <collision>
-        <origin xyz="0 -15.9e-3 28.35e-3" rpy="${-pi/6} 0 0" />
-        <geometry>
-          <box size="17.5e-3 7e-3 23.5e-3" />
-        </geometry>
-      </collision>
+      <xacro:if value="${collision_enable}">
+        <!-- screw mount -->
+        <collision>
+          <origin xyz="0 -18.5e-3 11e-3" rpy="0 0 0" />
+          <geometry>
+            <box size="22e-3 15e-3 20e-3" />
+          </geometry>
+        </collision>
+        <!-- cartriage sledge -->
+        <collision>
+          <origin xyz="0 -6.8e-3 2.2e-3" rpy="0 0 0" />
+          <geometry>
+            <box size="22e-3 8.8e-3 3.8e-3" />
+          </geometry>
+        </collision>
+        <!-- diagonal finger -->
+        <collision>
+          <origin xyz="0 -15.9e-3 28.35e-3" rpy="${-pi/6} 0 0" />
+          <geometry>
+            <box size="17.5e-3 7e-3 23.5e-3" />
+          </geometry>
+        </collision>
+      </xacro:if>
       <!-- rubber tip with which to grasp -->
       <collision>
@@ -114,5 +118,5 @@
       <axis xyz="0 -1 0" />
       <limit effort="100" lower="0.0" upper="0.04" velocity="0.2" />
-      <mimic joint="${arm_id}_finger_joint1" />
+      <!-- <mimic joint="${arm_id}_finger_joint1" /> -->
       <dynamics damping="0.3" />
     </joint>

File: panda_description/urdf/panda_robot.xacro (robot description, xacro)
@@ -1,5 +1,5 @@
 <?xml version='1.0' encoding='utf-8'?>
 <robot xmlns:xacro="http://www.ros.org/wiki/xacro">
-  <xacro:macro name="panda_robot" params="arm_id joint_limits hand gazebo ros2_control">
+  <xacro:macro name="panda_robot" params="arm_id joint_limits hand gazebo ros2_control collision_enable">
     <!-- Name of this panda -->
     <!-- Positional offset between $(arm_id)_hand -> $(arm_id)_hand_tcp [m]. Only used when hand:=true -->
@@ -9,5 +9,5 @@
     <xacro:include filename="$(find panda_description)/urdf/utils.xacro" />
     <xacro:include filename="$(find panda_description)/urdf/panda_arm.xacro" />
-    <xacro:panda_arm arm_id="${arm_id}" safety_distance="0.03" gazebo="$(arg gazebo)" joint_limits="${joint_limits}"/>
+    <xacro:panda_arm arm_id="${arm_id}" safety_distance="0.03" gazebo="$(arg gazebo)" joint_limits="${joint_limits}" collision_enable="${collision_enable}"/>
     <xacro:if value="$(arg hand)">
       <xacro:include filename="$(find panda_description)/urdf/panda_hand.xacro"/>
@@ -20,4 +20,5 @@
           safety_distance="0.03"
           gazebo="$(arg gazebo)"
+          collision_enable="${collision_enable}"
        />
     </xacro:if>

File: panda_description/urdf/utils.xacro (robot description, xacro)
@@ -33,5 +33,5 @@
   <!-- self_collision_geometries:  self <collision> models        -->
   <!-- ========================================================== -->
-  <xacro:macro name="link_with_sc" params="name prefix=${arm_id}_ rpy:='0 0 0' **self_collision_geometries gazebo:=false">
+  <xacro:macro name="link_with_sc" params="name prefix=${arm_id}_ rpy:='0 0 0' **self_collision_geometries gazebo:=false collision_enable:=true">
     <!-- sub-link defining detailed meshes for collision with environment -->
     <link name="${prefix}${name}">
@@ -42,7 +42,9 @@
       </visual>
       <collision>
-        <geometry>
-          <mesh filename="package://panda_description/meshes/collision/${name}.stl" />
-        </geometry>
+        <xacro:if value="${collision_enable}">
+          <geometry>
+            <mesh filename="package://panda_description/meshes/collision/${name}.stl" />
+          </geometry>
+        </xacro:if>
       </collision>
       <xacro:if value="${gazebo}">
