Commit message: 2.041 Updated the controllre parameters and sdf to remove the mimic joint of finger and include it as an independent joint

File: panda_moveit_config/config/panda.ros2_control.xacro (robot description, xacro)
@@ -2,5 +2,5 @@
 <robot xmlns:xacro="http://www.ros.org/wiki/xacro">
     <xacro:macro name="panda_ros2_control" params="name initial_positions_file">
-        <xacro:property name="initial_positions" value="${load_yaml(initial_positions_file)['initial_positions']}"/>
+        <xacro:property name="initial_positions" value="${xacro.load_yaml(initial_positions_file)['initial_positions']}"/>
         <ros2_control name="GazeboSystem" type="system">
             <hardware>
@@ -13,4 +13,5 @@
                 </state_interface>
                 <state_interface name="velocity"/>
+                <state_interface name="effort"/>
             </joint>
             <joint name="panda_joint2">
@@ -20,4 +21,5 @@
                 </state_interface>
                 <state_interface name="velocity"/>
+                <state_interface name="effort"/>
             </joint>
             <joint name="panda_joint3">
@@ -27,4 +29,5 @@
                 </state_interface>
                 <state_interface name="velocity"/>
+                <state_interface name="effort"/>
             </joint>
             <joint name="panda_joint4">
@@ -34,4 +37,5 @@
                 </state_interface>
                 <state_interface name="velocity"/>
+                <state_interface name="effort"/>
             </joint>
             <joint name="panda_joint5">
@@ -41,4 +45,5 @@
                 </state_interface>
                 <state_interface name="velocity"/>
+                <state_interface name="effort"/>
             </joint>
             <joint name="panda_joint6">
@@ -48,4 +53,5 @@
                 </state_interface>
                 <state_interface name="velocity"/>
+                <state_interface name="effort"/>
             </joint>
             <joint name="panda_joint7">
@@ -55,4 +61,5 @@
                 </state_interface>
                 <state_interface name="velocity"/>
+                <state_interface name="effort"/>
             </joint>
             <joint name="panda_finger_joint1">
@@ -62,4 +69,13 @@
                 </state_interface>
                 <state_interface name="velocity"/>
+                <state_interface name="effort"/>
+            </joint>
+            <joint name="panda_finger_joint2">
+                <command_interface name="position"/>
+                <state_interface name="position">
+                  <param name="initial_value">${initial_positions['panda_finger_joint2']}</param>
+                </state_interface>
+                <state_interface name="velocity"/>
+                <state_interface name="effort"/>
             </joint>
         </ros2_control>

File: panda_moveit_config/config/panda.urdf.xacro (robot description, xacro)
@@ -3,4 +3,5 @@
     <xacro:arg name="initial_positions_file" default="initial_positions.yaml" />
     <xacro:arg name="ros2_control" default="false" />
+    <xacro:arg name="collision_enable" default="false" />
     <!-- Import panda urdf file -->
     <xacro:include filename="$(find panda_description)/urdf/panda.urdf.xacro" />
